File: buzzer_circut.kicad_sch (KiCad schematic)
At the start: 4 parts, among them Q1 BC817-40-HT

Commit message: final design.
Parts:
- Q1: value BC817-40-HT -> BC807-40-HT; OZDISAN BC817-40-HT -> BC807-40-HT; özdisan BC817-40-HT -> BC807-40-HT
- renumbered D1 to D2, R14 to R21
Changed lines of the file:
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@@
 		(dnp no)
 		(fields_autoplaced yes)
-		(property "Reference" "#PWR049"
+		(property "Reference" "#PWR057"
 			(at 138.43 71.12 0)
 			(effects
@@
 			(project "mini_power_logger"
 				(path "/d0f26e02-819b-4fb4-bb3f-57422d098177/47813d3f-6b92-4c07-90fc-07f8d9e5daae"
-					(reference "#PWR049")
+					(reference "#PWR057")
 					(unit 1)
 				)
@@
 		(on_board yes)
 		(dnp no)
-		(property "Reference" "D1"
+		(property "Reference" "D2"
 			(at 134.62 73.3424 90)
 			(effects
@@
 			(project "mini_power_logger"
 				(path "/d0f26e02-819b-4fb4-bb3f-57422d098177/47813d3f-6b92-4c07-90fc-07f8d9e5daae"
-					(reference "D1")
+					(reference "D2")
 					(unit 1)
 				)
@@
 		(on_board yes)
 		(dnp no)
-		(property "Reference" "R14"
+		(property "Reference" "R21"
 			(at 128.524 83.058 90)
 			(effects
@@
 			(project "mini_power_logger"
 				(path "/d0f26e02-819b-4fb4-bb3f-57422d098177/47813d3f-6b92-4c07-90fc-07f8d9e5daae"
-					(reference "R14")
+					(reference "R21")
 					(unit 1)
 				)
@@
 		(on_board yes)
 		(dnp no)
-		(property "Reference" "#PWR050"
+		(property "Reference" "#PWR058"
 			(at 138.43 101.6 0)
 			(effects
@@
 			(project "mini_power_logger"
 				(path "/d0f26e02-819b-4fb4-bb3f-57422d098177/47813d3f-6b92-4c07-90fc-07f8d9e5daae"
-					(reference "#PWR050")
+					(reference "#PWR058")
 					(unit 1)
 				)
@@
 			)
 		)
-		(property "Value" "BC817-40-HT"
+		(property "Value" "BC807-40-HT"
 			(at 140.208 88.646 0)
 			(effects
@@
 			)
 		)
-		(property "OZDISAN" "BC817-40-HT"
+		(property "OZDISAN" "BC807-40-HT  "
 			(at 135.89 87.63 0)
 			(effects
@@
 			)
 		)
-		(property "özdisan" "BC817-40-HT"
+		(property "özdisan" "BC807-40-HT  "
 			(at 135.89 87.63 0)
 			(effects
