File: mini_power_logger.kicad_pcb (KiCad board)
At the start: 4 copper layers, 40 x 56 mm, 83 parts, among them J1 691322310002, J1 Screw_Terminal_01x03, J2 Screw_Terminal_01x02, J3 Screw_Terminal_01x02, J4 Conn_01x04_Pin, J5 Conn_01x02_Pin, J6 10k NTC Connector, J7 10k NTC Connector, J8 USB_C_Receptacle_USB2.0, P1 ST-TF-003A, L-KLS1-TF-003, Q1 BC817-40-HT, SW1 SW_Push, SW2 SW_Push, SW3 SW_Push, SW4 SW_Push, U1 STM32F103C8T6, U2 INA228, U3 OPA2197xD, U4 DM-OLED096-636, U5 TPS54302, Y1 AB26T-32.768KHZ-6, Y2 XD8M000000S418

Commit message: final design.
Parts:
- added G***: LOGO, footprints:mergened_footprints2.pretty, B.Cu at (177.7, 104.8)
Routing:
- net GND: track 35.8 -> 70.0 mm, vias 43 -> 55
- net /Type C Connector/USB2_P: track 47.9 -> 40.7 mm
- net /Type C Connector/USB2_N: track 47.9 -> 41.7 mm
