File: mini_power_logger.kicad_sch (KiCad schematic)
At the start: 4 parts, among them J1 Screw_Terminal_01x03, J2 Screw_Terminal_01x02, J3 Screw_Terminal_01x02

Commit message: final design.
Parts:
- J1, J2, J3: now not fitted
- J4: renamed from C1; now not fitted
Changed lines of the file:
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@@
 		(in_bom yes)
 		(on_board yes)
-		(dnp no)
-		(property "Reference" "C1"
+		(dnp yes)
+		(property "Reference" "J4"
 			(at 163.83 147.3199 0)
 			(effects
@@
 			(project ""
 				(path "/d0f26e02-819b-4fb4-bb3f-57422d098177"
-					(reference "C1")
+					(reference "J4")
 					(unit 1)
 				)
@@
 		(in_bom yes)
 		(on_board yes)
-		(dnp no)
+		(dnp yes)
 		(fields_autoplaced yes)
 		(property "Reference" "J2"
@@
 		(in_bom yes)
 		(on_board yes)
-		(dnp no)
+		(dnp yes)
 		(property "Reference" "J1"
 			(at 52.07 75.184 0)
@@
 		(in_bom yes)
 		(on_board yes)
-		(dnp no)
+		(dnp yes)
 		(fields_autoplaced yes)
 		(property "Reference" "J3"
