File: power.kicad_sch (KiCad schematic)
At the start: 14 parts, among them U5 TPS54302

Commit message: final design.
Parts:
- C21: renamed from C22; özdisan CC0603KRX7R9BB104 -> CC0603KRX7R9BB104
- C22: renamed from C23; özdisan CC0603KRX7R9BB104 -> CC0603KRX7R9BB104
- R18: renamed from R19; özdisan 0603SAF1332T5E -> 0603SAF2212T5E
- renumbered C21 to C20, C24 to C23, C25 to C24, C26 to C25, D2 to D1, R15 to R14, R16 to R15, R17 to R16, R18 to R17
Changed lines of the file:
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@@
 		(dnp no)
 		(fields_autoplaced yes)
-		(property "Reference" "R18"
+		(property "Reference" "R17"
 			(at 198.12 66.0399 0)
 			(effects
@@
 			(project "mini_power_logger"
 				(path "/d0f26e02-819b-4fb4-bb3f-57422d098177/672b4a3e-2ed1-44db-bfc6-31edf94eeab3"
-					(reference "R18")
+					(reference "R17")
 					(unit 1)
 				)
@@
 		(on_board yes)
 		(dnp no)
-		(property "Reference" "C25"
+		(property "Reference" "C24"
 			(at 183.134 57.912 0)
 			(effects
@@
 			(project "mini_power_logger"
 				(path "/d0f26e02-819b-4fb4-bb3f-57422d098177/672b4a3e-2ed1-44db-bfc6-31edf94eeab3"
-					(reference "C25")
+					(reference "C24")
 					(unit 1)
 				)
@@
 		(on_board yes)
 		(dnp no)
-		(property "Reference" "C26"
+		(property "Reference" "C25"
 			(at 190.754 65.532 0)
 			(effects
@@
 			(project "mini_power_logger"
 				(path "/d0f26e02-819b-4fb4-bb3f-57422d098177/672b4a3e-2ed1-44db-bfc6-31edf94eeab3"
-					(reference "C26")
+					(reference "C25")
 					(unit 1)
 				)
@@
 		(dnp no)
 		(fields_autoplaced yes)
-		(property "Reference" "#PWR053"
+		(property "Reference" "#PWR051"
 			(at 175.26 71.12 0)
 			(effects
@@
 			(project "mini_power_logger"
 				(path "/d0f26e02-819b-4fb4-bb3f-57422d098177/672b4a3e-2ed1-44db-bfc6-31edf94eeab3"
-					(reference "#PWR053")
+					(reference "#PWR051")
 					(unit 1)
 				)
@@
 		(dnp no)
 		(fields_autoplaced yes)
-		(property "Reference" "R17"
+		(property "Reference" "R16"
 			(at 198.12 58.4199 0)
 			(effects
@@
 			(project "mini_power_logger"
 				(path "/d0f26e02-819b-4fb4-bb3f-57422d098177/672b4a3e-2ed1-44db-bfc6-31edf94eeab3"
-					(reference "R17")
+					(reference "R16")
 					(unit 1)
 				)
@@
 		(on_board yes)
 		(dnp no)
-		(property "Reference" "C23"
+		(property "Reference" "C22"
 			(at 152.908 47.498 90)
 			(effects
@@
 			)
 		)
-		(property "özdisan" "CC0603KRX7R9BB104"
+		(property "özdisan" "CC0603KRX7R9BB104 "
 			(at 154.94 49.53 90)
 			(effects
@@
 			(project "mini_power_logger"
 				(path "/d0f26e02-819b-4fb4-bb3f-57422d098177/672b4a3e-2ed1-44db-bfc6-31edf94eeab3"
-					(reference "C23")
+					(reference "C22")
 					(unit 1)
 				)
@@
 		(dnp no)
 		(fields_autoplaced yes)
-		(property "Reference" "#PWR051"
+		(property "Reference" "#PWR049"
 			(at 96.52 82.55 0)
 			(effects
@@
 			(project "mini_power_logger"
 				(path "/d0f26e02-819b-4fb4-bb3f-57422d098177/672b4a3e-2ed1-44db-bfc6-31edf94eeab3"
-					(reference "#PWR051")
+					(reference "#PWR049")
 					(unit 1)
 				)
@@
 		(on_board yes)
 		(dnp no)
-		(property "Reference" "C21"
+		(property "Reference" "C20"
 			(at 98.044 59.69 0)
 			(effects
@@
 			(project "mini_power_logger"
 				(path "/d0f26e02-819b-4fb4-bb3f-57422d098177/672b4a3e-2ed1-44db-bfc6-31edf94eeab3"
-					(reference "C21")
+					(reference "C20")
 					(unit 1)
 				)
@@
 		(dnp no)
 		(fields_autoplaced yes)
-		(property "Reference" "#PWR055"
+		(property "Reference" "#PWR053"
 			(at 195.58 86.36 0)
 			(effects
@@
 			(project "mini_power_logger"
 				(path "/d0f26e02-819b-4fb4-bb3f-57422d098177/672b4a3e-2ed1-44db-bfc6-31edf94eeab3"
-					(reference "#PWR055")
+					(reference "#PWR053")
 					(unit 1)
 				)
@@
 		(on_board yes)
 		(dnp no)
-		(property "Reference" "R16"
+		(property "Reference" "R15"
 			(at 116.332 66.802 0)
 			(effects
@@
 			(project "mini_power_logger"
 				(path "/d0f26e02-819b-4fb4-bb3f-57422d098177/672b4a3e-2ed1-44db-bfc6-31edf94eeab3"
-					(reference "R16")
+					(reference "R15")
 					(unit 1)
 				)
@@
 		(dnp no)
 		(fields_autoplaced yes)
-		(property "Reference" "D2"
+		(property "Reference" "D1"
 			(at 91.44 45.72 0)
 			(effects
@@
 			(project "mini_power_logger"
 				(path "/d0f26e02-819b-4fb4-bb3f-57422d098177/672b4a3e-2ed1-44db-bfc6-31edf94eeab3"
-					(reference "D2")
+					(reference "D1")
 					(unit 1)
 				)
@@
 		(on_board yes)
 		(dnp no)
-		(property "Reference" "R19"
+		(property "Reference" "R18"
 			(at 198.12 73.6599 0)
 			(effects
@@
 			)
 		)
-		(property "özdisan" "0603SAF1332T5E"
+		(property "özdisan" "0603SAF2212T5E"
 			(at 195.58 74.93 0)
 			(effects
@@
 			(project "mini_power_logger"
 				(path "/d0f26e02-819b-4fb4-bb3f-57422d098177/672b4a3e-2ed1-44db-bfc6-31edf94eeab3"
-					(reference "R19")
+					(reference "R18")
 					(unit 1)
 				)
@@
 		(on_board yes)
 		(dnp no)
-		(property "Reference" "C24"
+		(property "Reference" "C23"
 			(at 169.926 57.658 0)
 			(effects
@@
 			(project "mini_power_logger"
 				(path "/d0f26e02-819b-4fb4-bb3f-57422d098177/672b4a3e-2ed1-44db-bfc6-31edf94eeab3"
-					(reference "C24")
+					(reference "C23")
 					(unit 1)
 				)
@@
 		(on_board yes)
 		(dnp no)
-		(property "Reference" "C22"
+		(property "Reference" "C21"
 			(at 106.426 59.436 0)
 			(effects
@@
 			)
 		)
-		(property "özdisan" "CC0603KRX7R9BB104"
+		(property "özdisan" "CC0603KRX7R9BB104 "
 			(at 105.41 62.23 0)
 			(effects
@@
 			(project "mini_power_logger"
 				(path "/d0f26e02-819b-4fb4-bb3f-57422d098177/672b4a3e-2ed1-44db-bfc6-31edf94eeab3"
-					(reference "C22")
+					(reference "C21")
 					(unit 1)
 				)
@@
 		(on_board yes)
 		(dnp no)
-		(property "Reference" "R15"
+		(property "Reference" "R14"
 			(at 115.824 56.642 0)
 			(effects
@@
 			(project "mini_power_logger"
 				(path "/d0f26e02-819b-4fb4-bb3f-57422d098177/672b4a3e-2ed1-44db-bfc6-31edf94eeab3"
-					(reference "R15")
+					(reference "R14")
 					(unit 1)
 				)
@@
 		(dnp no)
 		(fields_autoplaced yes)
-		(property "Reference" "#PWR052"
+		(property "Reference" "#PWR050"
 			(at 137.16 76.2 0)
 			(effects
@@
 			(project "mini_power_logger"
 				(path "/d0f26e02-819b-4fb4-bb3f-57422d098177/672b4a3e-2ed1-44db-bfc6-31edf94eeab3"
-					(reference "#PWR052")
+					(reference "#PWR050")
 					(unit 1)
 				)
@@
 		(dnp no)
 		(fields_autoplaced yes)
-		(property "Reference" "#PWR054"
+		(property "Reference" "#PWR052"
 			(at 195.58 58.42 0)
 			(effects
@@
 			(project "mini_power_logger"
 				(path "/d0f26e02-819b-4fb4-bb3f-57422d098177/672b4a3e-2ed1-44db-bfc6-31edf94eeab3"
-					(reference "#PWR054")
-					(unit 1)
-				)
+					(reference "#PWR052")
+					(unit 1)
+				)
