File: sd_card_spi.kicad_sch (KiCad schematic)
At the start: 2 parts, among them P1 ST-TF-003A, L-KLS1-TF-003, U4 DM-OLED096-636

Commit message: final design.
Parts:
- U4: now not fitted
Changed lines of the file:
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@@
 		(in_bom yes)
 		(on_board yes)
-		(dnp no)
+		(dnp yes)
 		(fields_autoplaced yes)
 		(property "Reference" "U4"
