File: sensors.kicad_sch (KiCad schematic)
At the start: 17 parts, among them J6 10k NTC Connector, J7 10k NTC Connector, U2 INA228, U3 OPA2197xD

Commit message: final design.
Parts:
- J7: renamed from J6; now not fitted
- J8: renamed from J7; now not fitted
- renumbered C16 to C15, C17 to C16, C18 to C17, C19 to C18, C20 to C19
Changed lines of the file:
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@@
 		(in_bom yes)
 		(on_board yes)
-		(dnp no)
-		(property "Reference" "J6"
+		(dnp yes)
+		(property "Reference" "J7"
 			(at 55.626 37.592 90)
 			(effects
@@
 			(project ""
 				(path "/d0f26e02-819b-4fb4-bb3f-57422d098177/d00f736a-765f-4a24-9c13-c76d4dd8f90d"
-					(reference "J6")
+					(reference "J7")
 					(unit 1)
 				)
@@
 		(on_board yes)
 		(dnp no)
-		(property "Reference" "C18"
+		(property "Reference" "C17"
 			(at 103.124 97.79 0)
 			(effects
@@
 			(project "mini_power_logger"
 				(path "/d0f26e02-819b-4fb4-bb3f-57422d098177/d00f736a-765f-4a24-9c13-c76d4dd8f90d"
-					(reference "C18")
+					(reference "C17")
 					(unit 1)
 				)
@@
 		(on_board yes)
 		(dnp no)
-		(property "Reference" "C16"
+		(property "Reference" "C15"
 			(at 57.15 148.082 0)
 			(effects
@@
 			(project "mini_power_logger"
 				(path "/d0f26e02-819b-4fb4-bb3f-57422d098177/d00f736a-765f-4a24-9c13-c76d4dd8f90d"
-					(reference "C16")
+					(reference "C15")
 					(unit 1)
 				)
@@
 		(on_board yes)
 		(dnp no)
-		(property "Reference" "C20"
+		(property "Reference" "C19"
 			(at 147.574 100.33 0)
 			(effects
@@
 			(project "mini_power_logger"
 				(path "/d0f26e02-819b-4fb4-bb3f-57422d098177/d00f736a-765f-4a24-9c13-c76d4dd8f90d"
-					(reference "C20")
+					(reference "C19")
 					(unit 1)
 				)
@@
 		(in_bom yes)
 		(on_board yes)
-		(dnp no)
-		(property "Reference" "J7"
+		(dnp yes)
+		(property "Reference" "J8"
 			(at 55.626 96.012 90)
 			(effects
@@
 			(project "mini_power_logger"
 				(path "/d0f26e02-819b-4fb4-bb3f-57422d098177/d00f736a-765f-4a24-9c13-c76d4dd8f90d"
-					(reference "J7")
+					(reference "J8")
 					(unit 1)
 				)
@@
 		(on_board yes)
 		(dnp no)
-		(property "Reference" "C17"
+		(property "Reference" "C16"
 			(at 103.124 39.37 0)
 			(effects
@@
 			(project "mini_power_logger"
 				(path "/d0f26e02-819b-4fb4-bb3f-57422d098177/d00f736a-765f-4a24-9c13-c76d4dd8f90d"
-					(reference "C17")
+					(reference "C16")
 					(unit 1)
 				)
@@
 		(on_board yes)
 		(dnp no)
-		(property "Reference" "C19"
+		(property "Reference" "C18"
 			(at 147.574 41.91 0)
 			(effects
@@
 			(project "mini_power_logger"
 				(path "/d0f26e02-819b-4fb4-bb3f-57422d098177/d00f736a-765f-4a24-9c13-c76d4dd8f90d"
-					(reference "C19")
-					(unit 1)
-				)
+					(reference "C18")
+					(unit 1)
+				)
