File: stm32f103c8t6.kicad_sch.kicad_sch (KiCad schematic)
At the start: 28 parts, among them J4 Conn_01x04_Pin, J5 Conn_01x02_Pin, SW1 SW_Push, SW2 SW_Push, SW3 SW_Push, SW4 SW_Push, U1 STM32F103C8T6, Y1 AB26T-32.768KHZ-6, Y2 XD8M000000S418

Commit message: final design.
Parts:
- J5: renamed from J4; now not fitted
- J6: renamed from J5; now not fitted
- renumbered C2 to C1, C11 to C10, C12 to C11, C13 to C12, C14 to C13, C15 to C14, C3 to C2, C4 to C3, C5 to C4, C6 to C5, C7 to C6, C8 to C7, C9 to C8, C10 to C9
Changed lines of the file:
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@@
 		(on_board yes)
 		(dnp no)
-		(property "Reference" "C12"
+		(property "Reference" "C11"
 			(at 155.194 119.126 0)
 			(effects
@@
 			(project "mini_power_logger"
 				(path "/d0f26e02-819b-4fb4-bb3f-57422d098177/7dc7dd08-c530-4987-bac3-6eaefc2cd844"
-					(reference "C12")
+					(reference "C11")
 					(unit 1)
 				)
@@
 		(on_board yes)
 		(dnp no)
-		(property "Reference" "C6"
+		(property "Reference" "C5"
 			(at 57.15 120.904 0)
 			(effects
@@
 			(project "mini_power_logger"
 				(path "/d0f26e02-819b-4fb4-bb3f-57422d098177/7dc7dd08-c530-4987-bac3-6eaefc2cd844"
-					(reference "C6")
+					(reference "C5")
 					(unit 1)
 				)
@@
 		(on_board yes)
 		(dnp no)
-		(property "Reference" "C5"
+		(property "Reference" "C4"
 			(at 55.6768 163.9316 0)
 			(effects
@@
 			(project "mini_power_logger"
 				(path "/d0f26e02-819b-4fb4-bb3f-57422d098177/7dc7dd08-c530-4987-bac3-6eaefc2cd844"
-					(reference "C5")
+					(reference "C4")
 					(unit 1)
 				)
@@
 		(in_bom yes)
 		(on_board yes)
-		(dnp no)
-		(property "Reference" "J4"
+		(dnp yes)
+		(property "Reference" "J5"
 			(at 25.908 89.154 0)
 			(effects
@@
 			(project "mini_power_logger"
 				(path "/d0f26e02-819b-4fb4-bb3f-57422d098177/7dc7dd08-c530-4987-bac3-6eaefc2cd844"
-					(reference "J4")
+					(reference "J5")
 					(unit 1)
 				)
@@
 		(on_board yes)
 		(dnp no)
-		(property "Reference" "C4"
+		(property "Reference" "C3"
 			(at 45.5168 163.9316 0)
 			(effects
@@
 			(project "mini_power_logger"
 				(path "/d0f26e02-819b-4fb4-bb3f-57422d098177/7dc7dd08-c530-4987-bac3-6eaefc2cd844"
-					(reference "C4")
+					(reference "C3")
 					(unit 1)
 				)
@@
 		(on_board yes)
 		(dnp no)
-		(property "Reference" "C7"
+		(property "Reference" "C6"
 			(at 65.8368 163.9316 0)
 			(effects
@@
 			(project "mini_power_logger"
 				(path "/d0f26e02-819b-4fb4-bb3f-57422d098177/7dc7dd08-c530-4987-bac3-6eaefc2cd844"
-					(reference "C7")
+					(reference "C6")
 					(unit 1)
 				)
@@
 		(on_board yes)
 		(dnp no)
-		(property "Reference" "C13"
+		(property "Reference" "C12"
 			(at 218.6432 34.1884 0)
 			(effects
@@
 			(project "mini_power_logger"
 				(path "/d0f26e02-819b-4fb4-bb3f-57422d098177/7dc7dd08-c530-4987-bac3-6eaefc2cd844"
-					(reference "C13")
+					(reference "C12")
 					(unit 1)
 				)
@@
 		(on_board yes)
 		(dnp no)
-		(property "Reference" "C15"
+		(property "Reference" "C14"
 			(at 218.6432 133.2484 0)
 			(effects
@@
 			(project "mini_power_logger"
 				(path "/d0f26e02-819b-4fb4-bb3f-57422d098177/7dc7dd08-c530-4987-bac3-6eaefc2cd844"
-					(reference "C15")
+					(reference "C14")
 					(unit 1)
 				)
@@
 		(on_board yes)
 		(dnp no)
-		(property "Reference" "C2"
+		(property "Reference" "C1"
 			(at 25.1968 163.9316 0)
 			(effects
@@
 			(project "mini_power_logger"
 				(path "/d0f26e02-819b-4fb4-bb3f-57422d098177/7dc7dd08-c530-4987-bac3-6eaefc2cd844"
-					(reference "C2")
+					(reference "C1")
 					(unit 1)
 				)
@@
 		(in_bom yes)
 		(on_board yes)
-		(dnp no)
-		(property "Reference" "J5"
+		(dnp yes)
+		(property "Reference" "J6"
 			(at 28.956 36.83 0)
 			(effects
@@
 			(project "mini_power_logger"
 				(path "/d0f26e02-819b-4fb4-bb3f-57422d098177/7dc7dd08-c530-4987-bac3-6eaefc2cd844"
-					(reference "J5")
+					(reference "J6")
 					(unit 1)
 				)
@@
 		(on_board yes)
 		(dnp no)
-		(property "Reference" "C8"
+		(property "Reference" "C7"
 			(at 74.7268 53.4416 0)
 			(effects
@@
 			(project "mini_power_logger"
 				(path "/d0f26e02-819b-4fb4-bb3f-57422d098177/7dc7dd08-c530-4987-bac3-6eaefc2cd844"
-					(reference "C8")
+					(reference "C7")
 					(unit 1)
 				)
@@
 		(on_board yes)
 		(dnp no)
-		(property "Reference" "C11"
+		(property "Reference" "C10"
 			(at 131.572 119.126 0)
 			(effects
@@
 			(project "mini_power_logger"
 				(path "/d0f26e02-819b-4fb4-bb3f-57422d098177/7dc7dd08-c530-4987-bac3-6eaefc2cd844"
-					(reference "C11")
+					(reference "C10")
 					(unit 1)
 				)
@@
 		(on_board yes)
 		(dnp no)
-		(property "Reference" "C10"
+		(property "Reference" "C9"
 			(at 81.0768 163.9316 0)
 			(effects
@@
 			(project "mini_power_logger"
 				(path "/d0f26e02-819b-4fb4-bb3f-57422d098177/7dc7dd08-c530-4987-bac3-6eaefc2cd844"
-					(reference "C10")
+					(reference "C9")
 					(unit 1)
 				)
@@
 		(on_board yes)
 		(dnp no)
-		(property "Reference" "C3"
+		(property "Reference" "C2"
 			(at 35.3568 163.9316 0)
 			(effects
@@
 			(project "mini_power_logger"
 				(path "/d0f26e02-819b-4fb4-bb3f-57422d098177/7dc7dd08-c530-4987-bac3-6eaefc2cd844"
-					(reference "C3")
+					(reference "C2")
 					(unit 1)
 				)
@@
 		(on_board yes)
 		(dnp no)
-		(property "Reference" "C14"
+		(property "Reference" "C13"
 			(at 218.6432 83.7184 0)
 			(effects
@@
 			(project "mini_power_logger"
 				(path "/d0f26e02-819b-4fb4-bb3f-57422d098177/7dc7dd08-c530-4987-bac3-6eaefc2cd844"
-					(reference "C14")
+					(reference "C13")
 					(unit 1)
 				)
@@
 		(on_board yes)
 		(dnp no)
-		(property "Reference" "C9"
+		(property "Reference" "C8"
 			(at 74.7268 120.7516 0)
 			(effects
@@
 			(project "mini_power_logger"
 				(path "/d0f26e02-819b-4fb4-bb3f-57422d098177/7dc7dd08-c530-4987-bac3-6eaefc2cd844"
-					(reference "C9")
+					(reference "C8")
 					(unit 1)
 				)
