File: usb_type_c.kicad_sch (KiCad schematic)
At the start: 5 parts, among them J8 USB_C_Receptacle_USB2.0

Commit message: final design.
Parts:
- renumbered C27 to C26, C28 to C27, J8 to J9, R20 to R19, R21 to R20
Changed lines of the file:
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@@
 		(dnp no)
 		(fields_autoplaced yes)
-		(property "Reference" "R21"
+		(property "Reference" "R20"
 			(at 186.69 100.3299 0)
 			(effects
@@
 			(project "mini_power_logger"
 				(path "/d0f26e02-819b-4fb4-bb3f-57422d098177/73ab6410-849a-425d-ad5e-08d2c341a4e9"
-					(reference "R21")
+					(reference "R20")
 					(unit 1)
 				)
@@
 		(dnp no)
 		(fields_autoplaced yes)
-		(property "Reference" "R20"
+		(property "Reference" "R19"
 			(at 173.99 100.3299 0)
 			(effects
@@
 			(project "mini_power_logger"
 				(path "/d0f26e02-819b-4fb4-bb3f-57422d098177/73ab6410-849a-425d-ad5e-08d2c341a4e9"
-					(reference "R20")
+					(reference "R19")
 					(unit 1)
 				)
@@
 		(on_board yes)
 		(dnp no)
-		(property "Reference" "C27"
+		(property "Reference" "C26"
 			(at 145.8468 97.8916 0)
 			(effects
@@
 			(project "mini_power_logger"
 				(path "/d0f26e02-819b-4fb4-bb3f-57422d098177/73ab6410-849a-425d-ad5e-08d2c341a4e9"
-					(reference "C27")
+					(reference "C26")
 					(unit 1)
 				)
@@
 		(on_board yes)
 		(dnp no)
-		(property "Reference" "C28"
+		(property "Reference" "C27"
 			(at 157.2768 97.8916 0)
 			(effects
@@
 			(project "mini_power_logger"
 				(path "/d0f26e02-819b-4fb4-bb3f-57422d098177/73ab6410-849a-425d-ad5e-08d2c341a4e9"
-					(reference "C28")
+					(reference "C27")
 					(unit 1)
 				)
@@
 		(dnp no)
 		(fields_autoplaced yes)
-		(property "Reference" "J8"
+		(property "Reference" "J9"
 			(at 118.11 59.69 0)
 			(effects
@@
 			(project "mini_power_logger"
 				(path "/d0f26e02-819b-4fb4-bb3f-57422d098177/73ab6410-849a-425d-ad5e-08d2c341a4e9"
-					(reference "J8")
+					(reference "J9")
 					(unit 1)
 				)
@@
 		(on_board yes)
 		(dnp no)
-		(property "Reference" "#PWR058"
+		(property "Reference" "#PWR056"
 			(at 177.8 114.3 0)
 			(effects
@@
 			(project "mini_power_logger"
 				(path "/d0f26e02-819b-4fb4-bb3f-57422d098177/73ab6410-849a-425d-ad5e-08d2c341a4e9"
-					(reference "#PWR058")
+					(reference "#PWR056")
 					(unit 1)
 				)
@@
 		(on_board yes)
 		(dnp no)
-		(property "Reference" "#PWR056"
+		(property "Reference" "#PWR054"
 			(at 114.3 113.03 0)
 			(effects
@@
 			(project "mini_power_logger"
 				(path "/d0f26e02-819b-4fb4-bb3f-57422d098177/73ab6410-849a-425d-ad5e-08d2c341a4e9"
-					(reference "#PWR056")
+					(reference "#PWR054")
 					(unit 1)
 				)
@@
 		(on_board yes)
 		(dnp no)
-		(property "Reference" "#PWR057"
+		(property "Reference" "#PWR055"
 			(at 143.51 111.76 0)
 			(effects
@@
 			(project "mini_power_logger"
 				(path "/d0f26e02-819b-4fb4-bb3f-57422d098177/73ab6410-849a-425d-ad5e-08d2c341a4e9"
-					(reference "#PWR057")
+					(reference "#PWR055")
 					(unit 1)
 				)
